Commit message: inference color change

File: objects/bigdustpan/bigdustpan.urdf (robot description, URDF)
Before this commit: robot smallbowl1, 1 links, 0 joints
Links:
- removed link smallbowl1
- added link bottle, mass 0.026; collision mesh filename=bigdustpan.obj scale=1.0 1.0 1.0; visual mesh filename=bigdustpan.obj scale=1.0 1.0 1.0

File: objects/bottle/bottle.urdf (robot description, URDF)
Before this commit: robot smallbowl1, 1 links, 0 joints
Links:
- removed link smallbowl1
- added link bottle, mass 0.2; collision mesh filename=bottle.obj scale=1.0 1.0 1.0; visual mesh filename=bottle.obj scale=1.0 1.0 1.0

File: objects/smallbowl1_inference/smallbowl1_inference.urdf (robot description, URDF)
Before this commit: robot smallbowl1, 1 links, 0 joints
Links:
- removed link smallbowl1
- added link smallbowl1_inference, mass 0.026; collision mesh filename=smallbowl1_inference.obj scale=1.0 1.0 1.0; visual mesh filename=smallbowl1_inference.obj scale=1.0 1.0 1.0
