Commit message: add root free version urdf

File: robots/hands/allegro_hand/allegro_hand_right_free.urdf (robot description, URDF)
Before this commit: robot allegro_hand_right, 29 links, 28 joints
Joints:
- joint x_joint: limit lower=-0.5 upper=0.5 effort=1 velocity=0 -> lower=-5.0 upper=5.0 effort=1 velocity=0
- joint y_joint: limit lower=-0.5 upper=0.5 effort=1 velocity=0 -> lower=-5.0 upper=5.0 effort=1 velocity=0
- joint z_joint: limit lower=-0.5 upper=0.5 effort=1 velocity=0 -> lower=-5.0 upper=5.0 effort=1 velocity=0

Commit message: update allegro

File: robots/hands/allegro_hand/allegro_hand_right_free.urdf (robot description, URDF)
Before this commit: robot allegro_hand_right, 29 links, 28 joints
Links:
- removed link palm_center
- added link wrist
- link base_link: geometry collision box size=0.0414 0.0538 0.0428; collision box size=0.0414 0.0720 0.013
- link link_0.0: mass 0.005 -> 0.0119
- link link_1.0: mass 0.125164 -> 0.065
- link link_10.0: mass 0.131691 -> 0.0355
- link link_11.0: mass 0.131691 -> 0.0096; geometry collision box size=0.0196 0.0269 0.022; visual mesh filename=meshes/visual/link_3.0.obj
- link link_11.0_tip: mass None -> 0.0168; geometry collision mesh filename=meshes/collision/link_tip.obj; visual mesh filename=meshes/visual/link_tip.obj
- link link_12.0: mass 0.005 -> 0.0176
- link link_13.0: mass 0.125164 -> 0.0119
- link link_14.0: mass 0.131691 -> 0.038
- link link_15.0: mass 0.131691 -> 0.0388; geometry collision box size=0.0196 0.0269 0.04; visual mesh filename=meshes/visual/link_15.0.obj
- link link_15.0_tip: mass None -> 0.0168; geometry collision mesh filename=meshes/collision/link_tip.obj; visual mesh filename=meshes/visual/link_tip.obj
- link link_2.0: mass 0.131691 -> 0.0355
- link link_3.0: mass 0.131691 -> 0.02; geometry collision box size=0.0196 0.0269 0.022; visual mesh filename=meshes/visual/link_3.0.obj
- link link_3.0_tip: mass None -> 0.0168; geometry collision mesh filename=meshes/collision/link_tip.obj; visual mesh filename=meshes/visual/link_tip.obj
- link link_5.0: mass 0.125164 -> 0.065
- link link_6.0: mass 0.131691 -> 0.0355
- link link_7.0: mass 0.131691 -> 0.0388; geometry collision box size=0.0196 0.0269 0.022; visual mesh filename=meshes/visual/link_3.0.obj
- link link_7.0_tip: mass None -> 0.0096; geometry collision mesh filename=meshes/collision/link_tip.obj; visual mesh filename=meshes/visual/link_tip.obj
- link link_9.0: mass 0.125164 -> 0.065
Joints:
- removed joint palm_center_joint
- added joint wrist_joint: type fixed, parent palm, child wrist, origin xyz=0 0 -0.03 rpy=0 0 0
- joint joint_0.0: limit lower=-0.47 upper=0.47 effort=10 velocity=0 -> lower=-0.47 upper=0.47 effort=10 velocity=3.14
- joint joint_1.0: limit lower=-0.196 upper=1.61 effort=10 velocity=0 -> lower=-0.196 upper=1.61 effort=10 velocity=3.14
- joint joint_10.0: limit lower=-0.174 upper=1.709 effort=10 velocity=0 -> lower=-0.174 upper=1.709 effort=10 velocity=3.14
- joint joint_11.0: limit lower=-0.227 upper=1.618 effort=10 velocity=0 -> lower=-0.227 upper=1.618 effort=10 velocity=3.14
- joint joint_12.0: limit lower=0.263 upper=1.396 effort=10 velocity=0 -> lower=0.263 upper=1.396 effort=10 velocity=3.14
- joint joint_13.0: limit lower=-0.105 upper=1.163 effort=10 velocity=0 -> lower=-0.105 upper=1.163 effort=10 velocity=3.14
- joint joint_14.0: limit lower=-0.189 upper=1.644 effort=10 velocity=0 -> lower=-0.189 upper=1.644 effort=10 velocity=3.14
- joint joint_15.0: limit lower=-0.162 upper=1.719 effort=10 velocity=0 -> lower=-0.162 upper=1.719 effort=10 velocity=3.14
- joint joint_2.0: limit lower=-0.174 upper=1.709 effort=10 velocity=0 -> lower=-0.174 upper=1.709 effort=10 velocity=3.14
- joint joint_3.0: limit lower=-0.227 upper=1.618 effort=10 velocity=0 -> lower=-0.227 upper=1.618 effort=10 velocity=3.14
- joint joint_4.0: limit lower=-0.47 upper=0.47 effort=10 velocity=0 -> lower=-0.47 upper=0.47 effort=10 velocity=3.14
- joint joint_5.0: limit lower=-0.196 upper=1.61 effort=10 velocity=0 -> lower=-0.196 upper=1.61 effort=10 velocity=3.14
- joint joint_6.0: limit lower=-0.174 upper=1.709 effort=10 velocity=0 -> lower=-0.174 upper=1.709 effort=10 velocity=3.14
- joint joint_7.0: limit lower=-0.227 upper=1.618 effort=10 velocity=0 -> lower=-0.227 upper=1.618 effort=10 velocity=3.14
- joint joint_8.0: limit lower=-0.47 upper=0.47 effort=10 velocity=0 -> lower=-0.47 upper=0.47 effort=10 velocity=3.14
- joint joint_9.0: limit lower=-0.196 upper=1.61 effort=10 velocity=0 -> lower=-0.196 upper=1.61 effort=10 velocity=3.14
- joint x_joint: limit lower=-5.0 upper=5.0 effort=1 velocity=0 -> lower=-50.0 upper=50.0 effort=1 velocity=0
- joint y_joint: limit lower=-5.0 upper=5.0 effort=1 velocity=0 -> lower=-50.0 upper=50.0 effort=1 velocity=0
- joint z_joint: limit lower=-5.0 upper=5.0 effort=1 velocity=0 -> lower=-50.0 upper=50.0 effort=1 velocity=0

Commit message: update

File: robots/hands/allegro_hand/allegro_hand_right_free.urdf (robot description, URDF)
Before this commit: robot allegro_right, 29 links, 28 joints
Joints:
- joint x_joint: limit lower=-50.0 upper=50.0 effort=1 velocity=0 -> lower=-50.0 upper=50.0 effort=100 velocity=0
- joint x_rotation_joint: limit lower=-3.14 upper=3.14 effort=1 velocity=0 -> lower=-6.28 upper=6.28 effort=100 velocity=0
- joint y_joint: limit lower=-50.0 upper=50.0 effort=1 velocity=0 -> lower=-50.0 upper=50.0 effort=100 velocity=0
- joint y_rotation_joint: limit lower=-3.14 upper=3.14 effort=1 velocity=0 -> lower=-6.28 upper=6.28 effort=100 velocity=0
- joint z_joint: limit lower=-50.0 upper=50.0 effort=1 velocity=0 -> lower=-50.0 upper=50.0 effort=100 velocity=0
- joint z_rotation_joint: limit lower=-3.14 upper=3.14 effort=1 velocity=0 -> lower=-6.28 upper=6.28 effort=100 velocity=0; origin xyz=0 0 0 rpy=-0.00000 -0.00000 0 -> (none)
