Commit message: inference color change

File: objects/book_inference/book_inference.urdf (robot description, URDF)
Before this commit: robot smallbowl1_inference, 1 links, 0 joints
Links:
- removed link smallbowl1_inference
- added link book_inference, mass 0.2; collision mesh filename=book_inference.obj scale=1.0 1.0 1.0; visual mesh filename=book_inference.obj scale=1.0 1.0 1.0

File: objects/bottle_inference/bottle_inference.urdf (robot description, URDF)
Before this commit: robot smallbowl1_inference, 1 links, 0 joints
Links:
- removed link smallbowl1_inference
- added link bottle_inference, mass 0.2; collision mesh filename=bottle_inference.obj scale=1.0 1.0 1.0; visual mesh filename=bottle_inference.obj scale=1.0 1.0 1.0
